Commit message: Blocked wrist-pitch and released prosupination

File: robot_models/icub/icubGazeboSim_fixedHeadWrist.urdf (robot description, URDF)
Before this commit: robot test_icub, 46 links, 45 joints
Joints:
- joint l_wrist_pitch: type revolute -> fixed
- joint l_wrist_prosup: type fixed -> revolute
- joint r_wrist_pitch: type revolute -> fixed
- joint r_wrist_prosup: type fixed -> revolute
