Commit message: Fixed bugs in URDF boxes computation Inserted Heron Formula Added torque check with RNEA Fixed bugs in rotation matrices

File: robot_models/threeLinkHumanLike/threeLinkHuman.urdf (robot description, URDF)
Before this commit: robot threeLinkHuman, 3 links, 2 joints
Joints:
- joint ankle: origin xyz=-0.025 0.0 0.05 rpy=0 0 0 -> xyz=-0.025 0 0.1 rpy=0 0 0
- joint hip: origin xyz=0.0 0.0 0.2 rpy=0 0 0 -> xyz=0 0 0.2 rpy=0 0 0
