Commit message: humanoids computations - several bugs squished

File: robot_models/threeLinkHumanLikeSubj3/threeLinkHuman_subject3.urdf (robot description, URDF)
Before this commit: robot threeLinkHuman_subject3, 3 links, 2 joints
Links:
- link foot: geometry collision box size=0.244 0.051 0.183; visual box size=0.244 0.051 0.183
- link leg: geometry collision box size=0.120 0.874 0.206; visual box size=0.120 0.874 0.206
- link torso: geometry collision box size=0.120 0.463 0.327; visual box size=0.120 0.463 0.327
Joints:
- joint ankle: axis 0 1 0 -> 0 0 1; origin xyz=-0.061 0 0.051 rpy=0 0 0 -> xyz=-0.061 -0.051 0 rpy=0 0 0
- joint hip: axis 0 1 0 -> 0 0 1; origin xyz=0 0 0.874 rpy=0 0 0 -> xyz=0 -0.874 0 rpy=0 0 0
