Commit message: modified script for creating for each subject the urdf file directly in the proper folder

File: human_models/threeLinkHumanLikeSubj01/threeLinkHuman_subject1.urdf (robot description, URDF)
Before this commit: robot threeLinkHuman, 3 links, 2 joints
Links:
- link foot: mass 3.0929 -> 3.0614; geometry collision box size=0.23091 0.12852 0.061354; visual box size=0.23091 0.12852 0.061354
- link leg: mass 25.5388 -> 25.4904; geometry collision box size=0.11545 0.16444 0.79851; visual box size=0.11545 0.16444 0.79851
- link torso: mass 33.0115 -> 33.1436; geometry collision box size=0.11545 0.31686 0.53883; visual box size=0.11545 0.31686 0.53883
Joints:
- joint ankle: origin xyz=-0.057733 0 0.061264 rpy=0 0 0 -> xyz=-0.057727 0 0.061354 rpy=0 0 0
- joint hip: origin xyz=0 0 0.79882 rpy=0 0 0 -> xyz=0 0 0.79851 rpy=0 0 0

File: human_models/threeLinkHumanLikeSubj02/threeLinkHuman_subject2.urdf (robot description, URDF)
Before this commit: robot threeLinkHuman_subject2, 3 links, 2 joints
Links:
- link foot: mass 4.3874 -> 4.3369; geometry collision box size=0.22229 0.21475 0.062401; visual box size=0.22229 0.21475 0.062401
- link leg: mass 30.6263 -> 30.6574; geometry collision box size=0.11115 0.23689 0.79975; visual box size=0.11115 0.23689 0.79975
- link torso: mass 28.6792 -> 28.5522; geometry collision box size=0.11115 0.35874 0.49184; visual box size=0.11115 0.35874 0.49184
Joints:
- joint ankle: origin xyz=-0.055533 0 0.063002 rpy=0 0 0 -> xyz=-0.055573 0 0.062401 rpy=0 0 0
- joint hip: origin xyz=0 0 0.7977 rpy=0 0 0 -> xyz=0 0 0.79975 rpy=0 0 0

File: human_models/threeLinkHumanLikeSubj03/threeLinkHuman_subject3.urdf (robot description, URDF)
Before this commit: robot threeLinkHuman_subject3, 3 links, 2 joints
Links:
- link foot: mass 4.754 -> 4.7562; geometry collision box size=0.22268 0.22544 0.062131; visual box size=0.22268 0.22544 0.062131
- link leg: mass 34.1044 -> 34.1076; geometry collision box size=0.11134 0.24976 0.80437; visual box size=0.11134 0.24976 0.80437
- link torso: mass 29.642 -> 29.6627; geometry collision box size=0.11134 0.3607 0.48437; visual box size=0.11134 0.3607 0.48437
Joints:
- joint ankle: origin xyz=-0.055704 0 0.062237 rpy=0 0 0 -> xyz=-0.055669 0 0.062131 rpy=0 0 0
- joint hip: origin xyz=0 0 0.80372 rpy=0 0 0 -> xyz=0 0 0.80437 rpy=0 0 0

File: human_models/threeLinkHumanLikeSubj04/threeLinkHuman_subject4.urdf (robot description, URDF)
Before this commit: robot threeLinkHuman_subject4, 3 links, 2 joints
Links:
- link foot: mass 4.3026 -> 4.2949; geometry collision box size=0.25991 0.15891 0.067446; visual box size=0.25991 0.15891 0.067446
- link leg: mass 37.3364 -> 37.3011; geometry collision box size=0.12996 0.20207 0.92131; visual box size=0.12996 0.20207 0.92131
- link torso: mass 35.4878 -> 35.4327; geometry collision box size=0.12996 0.35289 0.50114; visual box size=0.12996 0.35289 0.50114
Joints:
- joint ankle: origin xyz=-0.064958 0 0.067571 rpy=0 0 0 -> xyz=-0.064978 0 0.067446 rpy=0 0 0
- joint hip: origin xyz=0 0 0.92097 rpy=0 0 0 -> xyz=0 0 0.92131 rpy=0 0 0

File: human_models/threeLinkHumanLikeSubj05/threeLinkHuman_subject5.urdf (robot description, URDF)
Before this commit: robot threeLinkHuman_subject5, 3 links, 2 joints
Links:
- link foot: mass 4.2628 -> 4.2647; geometry collision box size=0.23637 0.20247 0.058784; visual box size=0.23637 0.20247 0.058784
- link leg: mass 31.6842 -> 31.7089; geometry collision box size=0.11819 0.21175 0.83581; visual box size=0.11819 0.21175 0.83581
- link torso: mass 27.1044 -> 27.1519; geometry collision box size=0.11819 0.29447 0.51466; visual box size=0.11819 0.29447 0.51466
Joints:
- joint ankle: origin xyz=-0.059093 0 0.0588 rpy=0 0 0 -> xyz=-0.059093 0 0.058784 rpy=0 0 0
- joint hip: origin xyz=0 0 0.83572 rpy=0 0 0 -> xyz=0 0 0.83581 rpy=0 0 0

File: human_models/threeLinkHumanLikeSubj06/threeLinkHuman_subject6.urdf (robot description, URDF)
Before this commit: robot threeLinkHuman_subject6, 3 links, 2 joints
Links:
- link foot: mass 4.0414 -> 4.0406; geometry collision box size=0.22693 0.21527 0.061164; visual box size=0.22693 0.21527 0.061164
- link leg: mass 32.706 -> 32.831; geometry collision box size=0.11347 0.2394 0.89374; visual box size=0.11347 0.2394 0.89374
- link torso: mass 20.1767 -> 20.0619; geometry collision box size=0.11347 0.29805 0.43867; visual box size=0.11347 0.29805 0.43867
Joints:
- joint ankle: origin xyz=-0.056785 0 0.061183 rpy=0 0 0 -> xyz=-0.056733 0 0.061164 rpy=0 0 0
- joint hip: origin xyz=0 0 0.89305 rpy=0 0 0 -> xyz=0 0 0.89374 rpy=0 0 0

File: human_models/threeLinkHumanLikeSubj07/threeLinkHuman_subject7.urdf (robot description, URDF)
Before this commit: robot threeLinkHuman_subject7, 3 links, 2 joints
Links:
- link foot: mass 4.3965 -> 4.3736; geometry collision box size=0.21591 0.18908 0.054016; visual box size=0.21591 0.18908 0.054016
- link leg: mass 32.1664 -> 32.0573; geometry collision box size=0.10795 0.20196 0.74134; visual box size=0.10795 0.20196 0.74134
- link torso: mass 35.7639 -> 35.5992; geometry collision box size=0.10795 0.32204 0.51627; visual box size=0.10795 0.32204 0.51627
Joints:
- joint ankle: origin xyz=-0.054021 0 0.053868 rpy=0 0 0 -> xyz=-0.053977 0 0.054016 rpy=0 0 0
- joint hip: origin xyz=0 0 0.7411 rpy=0 0 0 -> xyz=0 0 0.74134 rpy=0 0 0

File: human_models/threeLinkHumanLikeSubj08/threeLinkHuman_subject8.urdf (robot description, URDF)
Before this commit: robot threeLinkHuman_subject8, 3 links, 2 joints
Links:
- link foot: mass 6.7866 -> 6.7669; geometry collision box size=0.26372 0.29311 0.064746; visual box size=0.26372 0.29311 0.064746
- link leg: mass 41.4257 -> 41.4108; geometry collision box size=0.13186 0.28726 0.80859; visual box size=0.13186 0.28726 0.80859
- link torso: mass 35.2014 -> 35.2102; geometry collision box size=0.13186 0.36239 0.54497; visual box size=0.13186 0.36239 0.54497
Joints:
- joint ankle: origin xyz=-0.06587 0 0.064908 rpy=0 0 0 -> xyz=-0.06593 0 0.064746 rpy=0 0 0
- joint hip: origin xyz=0 0 0.80816 rpy=0 0 0 -> xyz=0 0 0.80859 rpy=0 0 0

File: human_models/threeLinkHumanLikeSubj09/threeLinkHuman_subject9.urdf (robot description, URDF)
Before this commit: robot threeLinkHuman_subject9, 3 links, 2 joints
Links:
- link foot: mass 5.0758 -> 5.1001; geometry collision box size=0.23505 0.27712 0.056924; visual box size=0.23505 0.27712 0.056924
- link leg: mass 35.6055 -> 35.397; geometry collision box size=0.11753 0.25877 0.84621; visual box size=0.11753 0.25877 0.84621
- link torso: mass 28.3345 -> 28.3864; geometry collision box size=0.11753 0.3544 0.49549; visual box size=0.11753 0.3544 0.49549
Joints:
- joint ankle: origin xyz=-0.058726 0 0.05673 rpy=0 0 0 -> xyz=-0.058763 0 0.056924 rpy=0 0 0
- joint hip: origin xyz=0 0 0.84702 rpy=0 0 0 -> xyz=0 0 0.84621 rpy=0 0 0

File: human_models/threeLinkHumanLikeSubj10/threeLinkHuman_subject10.urdf (robot description, URDF)
Before this commit: robot threeLinkHuman_subject10, 3 links, 2 joints
Links:
- link foot: mass 4.8692 -> 4.8865; geometry collision box size=0.23737 0.23741 0.062009; visual box size=0.23737 0.23741 0.062009
- link leg: mass 36.8554 -> 36.8533; geometry collision box size=0.11869 0.26871 0.82637; visual box size=0.11869 0.26871 0.82637
- link torso: mass 29.0139 -> 28.9449; geometry collision box size=0.11869 0.35385 0.49287; visual box size=0.11869 0.35385 0.49287
Joints:
- joint ankle: origin xyz=-0.05932 0 0.061803 rpy=0 0 0 -> xyz=-0.059343 0 0.062009 rpy=0 0 0
- joint hip: origin xyz=0 0 0.82696 rpy=0 0 0 -> xyz=0 0 0.82637 rpy=0 0 0

File: human_models/threeLinkHumanLikeSubj11/threeLinkHuman_subject11.urdf (robot description, URDF)
Before this commit: robot threeLinkHuman_subject11, 3 links, 2 joints
Links:
- link foot: mass 5.8636 -> 5.8868; geometry collision box size=0.2545 0.2436 0.070084; visual box size=0.2545 0.2436 0.070084
- link leg: mass 35.7206 -> 35.7058; geometry collision box size=0.12725 0.25714 0.80541; visual box size=0.12725 0.25714 0.80541
- link torso: mass 32.9495 -> 33.0867; geometry collision box size=0.12725 0.35456 0.54126; visual box size=0.12725 0.35456 0.54126
Joints:
- joint ankle: origin xyz=-0.063631 0 0.070188 rpy=0 0 0 -> xyz=-0.063625 0 0.070084 rpy=0 0 0
- joint hip: origin xyz=0 0 0.80566 rpy=0 0 0 -> xyz=0 0 0.80541 rpy=0 0 0

File: human_models/threeLinkHumanLikeSubj12/threeLinkHuman_subject12.urdf (robot description, URDF)
Before this commit: robot threeLinkHuman_subject12, 3 links, 2 joints
Links:
- link foot: mass 3.048 -> 3.0638; geometry collision box size=0.23416 0.1207 0.067347; visual box size=0.23416 0.1207 0.067347
- link leg: mass 28.1065 -> 28.0587; geometry collision box size=0.11708 0.18398 0.80928; visual box size=0.11708 0.18398 0.80928
- link torso: mass 32.6978 -> 32.7694; geometry collision box size=0.11708 0.33651 0.51673; visual box size=0.11708 0.33651 0.51673
Joints:
- joint ankle: origin xyz=-0.058581 0 0.067319 rpy=0 0 0 -> xyz=-0.058539 0 0.067347 rpy=0 0 0
- joint hip: origin xyz=0 0 0.80946 rpy=0 0 0 -> xyz=0 0 0.80928 rpy=0 0 0

Commit message: modifications for major review (finding the ground truth)

File: human_models/threeLinkHumanLikeSubj01/threeLinkHuman_subject1.urdf (robot description, URDF)
Before this commit: robot threeLinkHuman, 3 links, 2 joints
Links:
- link foot: mass 3.0614 -> 3.0639; geometry collision box size=0.23162 0.12793 0.061755; visual box size=0.23162 0.12793 0.061755
- link leg: mass 25.4904 -> 25.5563; geometry collision box size=0.11581 0.16536 0.79699; visual box size=0.11581 0.16536 0.79699
- link torso: mass 33.1436 -> 33.0707; geometry collision box size=0.11581 0.31673 0.53846; visual box size=0.11581 0.31673 0.53846
Joints:
- joint ankle: origin xyz=-0.057727 0 0.061354 rpy=0 0 0 -> xyz=-0.057906 0 0.061755 rpy=0 0 0
- joint hip: origin xyz=0 0 0.79851 rpy=0 0 0 -> xyz=0 0 0.79699 rpy=0 0 0

File: human_models/threeLinkHumanLikeSubj03/threeLinkHuman_subject3.urdf (robot description, URDF)
Before this commit: robot threeLinkHuman, 3 links, 2 joints
Links:
- link foot: mass 4.7562 -> 4.3179; geometry collision box size=0.22229 0.21638 0.061439; visual box size=0.22229 0.21638 0.061439
- link leg: mass 34.1076 -> 30.6242; geometry collision box size=0.11115 0.23449 0.80417; visual box size=0.11115 0.23449 0.80417
- link torso: mass 29.6627 -> 33.6115; geometry collision box size=0.11115 0.35851 0.49141; visual box size=0.11115 0.35851 0.49141
Joints:
- joint ankle: origin xyz=-0.055669 0 0.062131 rpy=0 0 0 -> xyz=-0.055573 0 0.061439 rpy=0 0 0
- joint hip: origin xyz=0 0 0.80437 rpy=0 0 0 -> xyz=0 0 0.80417 rpy=0 0 0

File: human_models/threeLinkHumanLikeSubj04/threeLinkHuman_subject4.urdf (robot description, URDF)
Before this commit: robot threeLinkHuman, 3 links, 2 joints
Links:
- link foot: mass 4.2949 -> 4.271; geometry collision box size=0.25948 0.16008 0.066806; visual box size=0.25948 0.16008 0.066806
- link leg: mass 37.3011 -> 37.5187; geometry collision box size=0.12974 0.20314 0.92497; visual box size=0.12974 0.20314 0.92497
- link torso: mass 35.4327 -> 35.2685; geometry collision box size=0.12974 0.35233 0.50131; visual box size=0.12974 0.35233 0.50131
Joints:
- joint ankle: origin xyz=-0.064978 0 0.067446 rpy=0 0 0 -> xyz=-0.064871 0 0.066806 rpy=0 0 0
- joint hip: origin xyz=0 0 0.92131 rpy=0 0 0 -> xyz=0 0 0.92497 rpy=0 0 0

File: human_models/threeLinkHumanLikeSubj05/threeLinkHuman_subject5.urdf (robot description, URDF)
Before this commit: robot threeLinkHuman, 3 links, 2 joints
Links:
- link foot: mass 4.2647 -> 4.2068; geometry collision box size=0.23584 0.20217 0.058416; visual box size=0.23584 0.20217 0.058416
- link leg: mass 31.7089 -> 31.9962; geometry collision box size=0.11792 0.21424 0.83853; visual box size=0.11792 0.21424 0.83853
- link torso: mass 27.1519 -> 26.9246; geometry collision box size=0.11792 0.294 0.51419; visual box size=0.11792 0.294 0.51419
Joints:
- joint ankle: origin xyz=-0.059093 0 0.058784 rpy=0 0 0 -> xyz=-0.058959 0 0.058416 rpy=0 0 0
- joint hip: origin xyz=0 0 0.83581 rpy=0 0 0 -> xyz=0 0 0.83853 rpy=0 0 0

File: human_models/threeLinkHumanLikeSubj06/threeLinkHuman_subject6.urdf (robot description, URDF)
Before this commit: robot threeLinkHuman, 3 links, 2 joints
Links:
- link foot: mass 4.0406 -> 4.0649; geometry collision box size=0.22694 0.21373 0.061353; visual box size=0.22694 0.21373 0.061353
- link leg: mass 32.831 -> 32.7484; geometry collision box size=0.11347 0.23703 0.8914; visual box size=0.11347 0.23703 0.8914
- link torso: mass 20.0619 -> 20.1525; geometry collision box size=0.11347 0.29848 0.43561; visual box size=0.11347 0.29848 0.43561
Joints:
- joint ankle: origin xyz=-0.056733 0 0.061164 rpy=0 0 0 -> xyz=-0.056735 0 0.061353 rpy=0 0 0
- joint hip: origin xyz=0 0 0.89374 rpy=0 0 0 -> xyz=0 0 0.8914 rpy=0 0 0

File: human_models/threeLinkHumanLikeSubj08/threeLinkHuman_subject8.urdf (robot description, URDF)
Before this commit: robot threeLinkHuman, 3 links, 2 joints
Links:
- link foot: mass 6.7669 -> 6.7414; geometry collision box size=0.26458 0.29375 0.06473; visual box size=0.26458 0.29375 0.06473
- link leg: mass 41.4108 -> 41.5446; geometry collision box size=0.13229 0.28966 0.80908; visual box size=0.13229 0.28966 0.80908
- link torso: mass 35.2102 -> 35.0679; geometry collision box size=0.13229 0.36273 0.54536; visual box size=0.13229 0.36273 0.54536
Joints:
- joint ankle: origin xyz=-0.06593 0 0.064746 rpy=0 0 0 -> xyz=-0.066145 0 0.06473 rpy=0 0 0
- joint hip: origin xyz=0 0 0.80859 rpy=0 0 0 -> xyz=0 0 0.80908 rpy=0 0 0

File: human_models/threeLinkHumanLikeSubj09/threeLinkHuman_subject9.urdf (robot description, URDF)
Before this commit: robot threeLinkHuman, 3 links, 2 joints
Links:
- link foot: mass 5.1001 -> 5.2252; geometry collision box size=0.235 0.27785 0.056733; visual box size=0.235 0.27785 0.056733
- link leg: mass 35.397 -> 34.7124; geometry collision box size=0.1175 0.24795 0.84469; visual box size=0.1175 0.24795 0.84469
- link torso: mass 28.3864 -> 28.9538; geometry collision box size=0.1175 0.35384 0.4937; visual box size=0.1175 0.35384 0.4937
Joints:
- joint ankle: origin xyz=-0.058763 0 0.056924 rpy=0 0 0 -> xyz=-0.058751 0 0.056733 rpy=0 0 0
- joint hip: origin xyz=0 0 0.84621 rpy=0 0 0 -> xyz=0 0 0.84469 rpy=0 0 0

File: human_models/threeLinkHumanLikeSubj10/threeLinkHuman_subject10.urdf (robot description, URDF)
Before this commit: robot threeLinkHuman, 3 links, 2 joints
Links:
- link foot: mass 4.8865 -> 4.8738; geometry collision box size=0.23861 0.23504 0.061603; visual box size=0.23861 0.23504 0.061603
- link leg: mass 36.8533 -> 36.3607; geometry collision box size=0.1193 0.2615 0.82618; visual box size=0.1193 0.2615 0.82618
- link torso: mass 28.9449 -> 29.345; geometry collision box size=0.1193 0.35413 0.49236; visual box size=0.1193 0.35413 0.49236
Joints:
- joint ankle: origin xyz=-0.059343 0 0.062009 rpy=0 0 0 -> xyz=-0.059652 0 0.061603 rpy=0 0 0
- joint hip: origin xyz=0 0 0.82637 rpy=0 0 0 -> xyz=0 0 0.82618 rpy=0 0 0

File: human_models/threeLinkHumanLikeSubj11/threeLinkHuman_subject11.urdf (robot description, URDF)
Before this commit: robot threeLinkHuman, 3 links, 2 joints
Links:
- link foot: mass 5.8868 -> 5.9204; geometry collision box size=0.25481 0.24345 0.070543; visual box size=0.25481 0.24345 0.070543
- link leg: mass 35.7058 -> 35.8194; geometry collision box size=0.1274 0.25833 0.80444; visual box size=0.1274 0.25833 0.80444
- link torso: mass 33.0867 -> 32.8776; geometry collision box size=0.1274 0.35418 0.53855; visual box size=0.1274 0.35418 0.53855
Joints:
- joint ankle: origin xyz=-0.063625 0 0.070084 rpy=0 0 0 -> xyz=-0.063702 0 0.070543 rpy=0 0 0
- joint hip: origin xyz=0 0 0.80541 rpy=0 0 0 -> xyz=0 0 0.80444 rpy=0 0 0

File: human_models/threeLinkHumanLikeSubj12/threeLinkHuman_subject12.urdf (robot description, URDF)
Before this commit: robot threeLinkHuman, 3 links, 2 joints
Links:
- link foot: mass 3.0638 -> 3.164; geometry collision box size=0.23351 0.12544 0.066979; visual box size=0.23351 0.12544 0.066979
- link leg: mass 28.0587 -> 28.0108; geometry collision box size=0.11676 0.18359 0.81032; visual box size=0.11676 0.18359 0.81032
- link torso: mass 32.7694 -> 32.724; geometry collision box size=0.11676 0.33676 0.51607; visual box size=0.11676 0.33676 0.51607
Joints:
- joint ankle: origin xyz=-0.058539 0 0.067347 rpy=0 0 0 -> xyz=-0.058378 0 0.066979 rpy=0 0 0
- joint hip: origin xyz=0 0 0.80928 rpy=0 0 0 -> xyz=0 0 0.81032 rpy=0 0 0

File: human_models/threeLinkHumanLikeSubj14/threeLinkHuman_subject14.urdf (robot description, URDF)
Before this commit: robot threeLinkHuman, 3 links, 2 joints
Links:
- link foot: mass 4.431 -> 0; geometry collision box size=0.22229 0.21638 0.061439; visual box size=0.22229 0.21638 0.061439
- link leg: mass 32.8563 -> 0; geometry collision box size=0.11115 0.23449 0.80417; visual box size=0.11115 0.23449 0.80417
- link torso: mass 36.0421 -> 5; geometry collision box size=0.11115 0.35851 0.49141; visual box size=0.11115 0.35851 0.49141
Joints:
- joint ankle: origin xyz=-0.053944 0 0.05465 rpy=0 0 0 -> xyz=-0.055573 0 0.061439 rpy=0 0 0
- joint hip: origin xyz=0 0 0.74003 rpy=0 0 0 -> xyz=0 0 0.80417 rpy=0 0 0
